File: impednace-analyzer-pcb/hardware/impedance-analyzer/impedance-analyzer.kicad_pcb (KiCad board)
At the start: 2 copper layers, 61.9 x 56.5 mm, 11 parts, among them J1 AD9833, J2 ADS1256_SPI, J3 ADS1256_AIN, J4 UNO_POWER, J5 UNO_ANALOG, J6 UNO_DIGITAL_LOW, J7 UNO_DIGITAL_HIGH, J8 PIEZO

Commit message: updated schematic
Parts:
- added J10: Conn_01x08, Connector_Molex:Molex_Micro-Fit_3.0_43650-0815_1x08_P3.00mm_Vertical, F.Cu at (197.3, 115.2)
- added J11: Conn_01x08, Connector_Molex:Molex_Micro-Fit_3.0_43650-0815_1x08_P3.00mm_Vertical, F.Cu at (197.3, 123.1)
- added J12: Conn_01x08, Connector_Molex:Molex_Micro-Fit_3.0_43650-0815_1x08_P3.00mm_Vertical, F.Cu at (197.3, 130.9)
- added J9: Conn_01x08, Connector_Molex:Molex_Micro-Fit_3.0_43650-0815_1x08_P3.00mm_Vertical, F.Cu at (197.3, 107.4)
- added R1: 10k, Resistor_SMD:R_0805_2012Metric_Pad1.20x1.40mm_HandSolder, F.Cu at (243.4, 92.0)
- added U1: CD74HC4067M, Package_DIP:DIP-24_W7.62mm, F.Cu at (225.6, 97.8)
- J8: value PIEZO -> Conn_01x08; footprint TerminalBlock:TerminalBlock_MaiXu_MX126-5.0-02P_1x02_P5.00mm -> Connector_Molex:Molex_Micro-Fit_3.0_43650-0815_1x08_P3.00mm_Vertical
- moved J1 69.5 mm to (200.3, 62.9)
- moved J8 32.2 mm to (197.3, 99.6)
- moved J3 0.21 mm to (227.0, 60.0)
Connections:
- J3 pad 1: AD9833_OUT -> GND
- J3 pad 10: unconnected-(J3-Pin_10-Pad10) -> GND
- J3 pad 11: unconnected-(J3-Pin_11-Pad11) -> GND
- J3 pad 12: unconnected-(J3-Pin_12-Pad12) -> GND
- J3 pad 13: unconnected-(J3-Pin_13-Pad13) -> GND
- J3 pad 14: unconnected-(J3-Pin_14-Pad14) -> GND
- J3 pad 2: GND -> AD9833_OUT
- J3 pad 3: VMID_NODE -> GND
- J3 pad 4: GND -> VMID_NODE
- J3 pad 5: unconnected-(J3-Pin_5-Pad5) -> GND
- J3 pad 6: unconnected-(J3-Pin_6-Pad6) -> GND
- J3 pad 7: unconnected-(J3-Pin_7-Pad7) -> GND
- J3 pad 8: unconnected-(J3-Pin_8-Pad8) -> GND
- J3 pad 9: unconnected-(J3-Pin_9-Pad9) -> GND
- J5 pad 1: unconnected-(J5-Pin_1-Pad1) -> DB_S1
- J5 pad 2: unconnected-(J5-Pin_2-Pad2) -> DB_S2
- J5 pad 3: unconnected-(J5-Pin_3-Pad3) -> DB_S3
- J5 pad 4: unconnected-(J5-Pin_4-Pad4) -> DB_EN
- J6 pad 3: unconnected-(J6-Pin_3-Pad3) -> MB_S0
- J6 pad 4: unconnected-(J6-Pin_4-Pad4) -> MB_S1
- J6 pad 5: unconnected-(J6-Pin_5-Pad5) -> MB_S2
- J6 pad 6: unconnected-(J6-Pin_6-Pad6) -> MB_S3
- J6 pad 7: unconnected-(J6-Pin_7-Pad7) -> MB_EN
- J6 pad 8: unconnected-(J6-Pin_8-Pad8) -> DB_S0
- J8 pad 1: VMID_NODE -> JACK0_SIG
