File: sensor-board-pcb/sensorboard/sensorboard.kicad_pcb (KiCad board)
At the start: 2 copper layers, 80 x 72 mm, 19 parts, among them J1 TO_MOTHERBOARD, J10 PZT_08, J11 PZT_09, J12 PZT_10, J13 PZT_11, J14 PZT_12, J15 PZT_13, J16 PZT_14, J17 PZT_15, J2 PZT_00, J3 PZT_01, J4 PZT_02, J5 PZT_03, J6 PZT_04, J7 PZT_05, J8 PZT_06, J9 PZT_07, U1 CD74HC4067M

Commit message: fixed schematic and finished routing
Parts:
- added R1: 10k, Resistor_THT:R_Axial_DIN0207_L6.3mm_D2.5mm_P7.62mm_Horizontal, F.Cu at (150.5, 97.8)
- C1: footprint Capacitor_SMD:C_0603_1608Metric -> Capacitor_THT:C_Disc_D5.0mm_W2.5mm_P5.00mm
- moved C1 8.50 mm to (140.0, 60.5), turned to 0 degrees
Connections:
- J1 pad 1: +5V -> ANALOG_COM
- J1 pad 2: ANALOG_COM -> GND
- J1 pad 3: GND -> DB_S0
- J1 pad 4: DB_S0 -> DB_S1
- J1 pad 5: DB_S1 -> DB_S2
- J1 pad 6: DB_S2 -> DB_S3
- J1 pad 7: DB_S3 -> DB_EN
- J1 pad 8: DB_EN -> +5V
- U1 pad 1: DB_EN -> ANALOG_COM
- U1 pad 10: DB_S3 -> DB_S0
- U1 pad 11: DB_S0 -> DB_S1
- U1 pad 13: DB_S2 -> DB_S3
- U1 pad 14: DB_S1 -> DB_S2
- U1 pad 15: ANALOG_COM -> DB_EN
Routing:
- net DB_EN: track 0.00 -> 53.6 mm, vias 0 -> 2
- net +5V: track 27.5 -> 80.9 mm, vias 0 -> 2
- net DB_S3: track 0.00 -> 52.8 mm, vias 0 -> 2
- net DB_S1: track 0.00 -> 50.2 mm, vias 0 -> 2
- net DB_S2: track 0.00 -> 49.9 mm, vias 0 -> 2
- net DB_S0: track 0.00 -> 44.3 mm, vias 0 -> 2
- net ANALOG_COM: track 0.00 -> 20.5 mm
- added copper zone on B.Cu, net GND
