File: single-sensor-pcb/impedance-analyzer.kicad_sch (KiCad schematic)
At the start: 11 parts, among them J1 AD9833, J2 ADS1256_SPI, J3 ADS1256_AIN, J4 UNO_POWER, J5 UNO_ANALOG, J6 UNO_DIGITAL_LOW, J7 UNO_DIGITAL_HIGH, J8 PIEZO

Commit message: routed single sensor board, drc clean
Parts:
- C1, C2: footprint Capacitor_SMD:C_0805_2012Metric_Pad1.18x1.45mm_HandSolder -> Capacitor_THT:C_Disc_D5.0mm_W2.5mm_P5.00mm
- J8: footprint TerminalBlock:TerminalBlock_MaiXu_MX126-5.0-02P_1x02_P5.00mm -> TerminalBlock_Phoenix:TerminalBlock_Phoenix_MPT-0,5-2-2.54_1x02_P2.54mm_Horizontal
Connections:
- net GND: now also J3.10 (Pin_10), J3.11 (Pin_11), J3.12 (Pin_12), J3.13 (Pin_13), J3.14 (Pin_14), J3.5 (Pin_5), J3.6 (Pin_6), J3.7 (Pin_7), J3.8 (Pin_8), J3.9 (Pin_9)
- no-connect marks 32 -> 22
